Commit message: Añadidos cambios para usar la cámara montable y cambiada la lógica de decisión de objetos de interés al nodo yolo

File: src/go2_ros2_sdk/src/go2_robot_sdk/urdf/go2_with_realsense.urdf (robot description, URDF)
Before this commit: robot go2, 35 links, 34 joints
Joints:
- joint camera_mount_joint: origin xyz=-0.0647 0 0.07 rpy=0 0 0 -> xyz=0.0357 0 0.03 rpy=0 0 0
- joint realsense_d435i_joint: origin xyz=0 0 0.0425 rpy=0 0.05 0 -> xyz=0.005 0 0.0425 rpy=0 0.25 0
